Commit message: Set limits in urdf

File: kuka_kr10_support/urdf/kr10r1100sixx_macro.xacro (robot description, xacro)
@@ -122,5 +122,5 @@
       <child link="${prefix}link_2"/>
       <axis xyz="0 1 0"/>
-      <limit effort="0" lower="${radians(-190)}" upper="${radians(45)}" velocity="${radians(225)}"/>
+      <limit effort="0" lower="${radians(-190)}" upper="${radians(0)}" velocity="${radians(225)}"/>
     </joint>
     <joint name="${prefix}joint_a3" type="revolute">
@@ -129,5 +129,5 @@
       <child link="${prefix}link_3"/>
       <axis xyz="0 1 0"/>
-      <limit effort="0" lower="${radians(-120)}" upper="${radians(156)}" velocity="${radians(225)}"/>
+      <limit effort="0" lower="${radians(0)}" upper="${radians(156)}" velocity="${radians(225)}"/>
     </joint>
     <joint name="${prefix}joint_a4" type="revolute">
@@ -136,5 +136,5 @@
       <child link="${prefix}link_4"/>
       <axis xyz="-1 0 0"/>
-      <limit effort="0" lower="${radians(-185)}" upper="${radians(185)}" velocity="${radians(381)}"/>
+      <limit effort="0" lower="${radians(-120)}" upper="${radians(120)}" velocity="${radians(381)}"/>
     </joint>
     <joint name="${prefix}joint_a5" type="revolute">
@@ -143,5 +143,5 @@
       <child link="${prefix}link_5"/>
       <axis xyz="0 1 0"/>
-      <limit effort="0" lower="${radians(-120)}" upper="${radians(120)}" velocity="${radians(311)}"/>
+      <limit effort="0" lower="${radians(0)}" upper="${radians(90)}" velocity="${radians(311)}"/>
     </joint>
     <joint name="${prefix}joint_a6" type="revolute">
@@ -150,5 +150,5 @@
       <child link="${prefix}link_6"/>
       <axis xyz="-1 0 0"/>
-      <limit effort="0" lower="${radians(-350)}" upper="${radians(350)}" velocity="${radians(492)}"/>
+      <limit effort="0" lower="${radians(-120)}" upper="${radians(120)}" velocity="${radians(492)}"/>
     </joint>
     <joint name="${prefix}joint_a6-flange" type="fixed">

Commit message: Dirtily updated colours

File: kuka_kr10_support/urdf/kr10r1100sixx_macro.xacro (robot description, xacro)
@@ -3,4 +3,5 @@
   <xacro:macro name="kuka_kr10r1100sixx" params="prefix">
     <xacro:include filename="$(find kuka_resources)/urdf/common_materials.xacro"/>
+    <xacro:include filename="$(find kuka_kr10_support)/urdf/kr10r1100sixx_macro.xacro" />
     <link name="${prefix}base_link">
       <visual>
@@ -9,5 +10,5 @@
           <mesh filename="package://kuka_kr10_support/meshes/kr10r1100sixx/visual/base_link.stl" />
         </geometry>
-        <xacro:material_kuka_black />
+        <material name="zed2i_mat"/>
       </visual>
       <collision>
@@ -24,5 +25,5 @@
           <mesh filename="package://kuka_kr10_support/meshes/kr10r1100sixx/visual/link_1.stl" />
         </geometry>
-        <xacro:material_kuka_orange />
+        <xacro:material_kuka_ral_pure_white />
       </visual>
       <collision>
@@ -39,5 +40,5 @@
           <mesh filename="package://kuka_kr10_support/meshes/kr10r1100sixx/visual/link_2.stl"/>
         </geometry>
-        <xacro:material_kuka_orange />
+        <xacro:material_kuka_ral_pure_white />
       </visual>
       <collision>
@@ -54,5 +55,5 @@
           <mesh filename="package://kuka_kr10_support/meshes/kr10r1100sixx/visual/link_3.stl" />
         </geometry>
-        <xacro:material_kuka_orange />
+        <xacro:material_kuka_ral_pure_white />
       </visual>
       <collision>
@@ -69,5 +70,5 @@
           <mesh filename="package://kuka_kr10_support/meshes/kr10r1100sixx/visual/link_4.stl" />
         </geometry>
-        <xacro:material_kuka_orange />
+        <xacro:material_kuka_ral_pure_white />
       </visual>
       <collision>
@@ -84,5 +85,5 @@
           <mesh filename="package://kuka_kr10_support/meshes/kr10r1100sixx/visual/link_5.stl" />
         </geometry>
-        <xacro:material_kuka_orange />
+        <xacro:material_kuka_ral_pure_white />
       </visual>
       <collision>
